File: electrical/BMS/BMS_vtest/BMS_vtest.kicad_pcb (KiCad board)
At the start: 4 copper layers, 116 parts, among them J1 Conn_01x04_Pin, J2 Conn_02x12_Top_Bottom, J3 Conn_01x13_Socket, J4 Conn_01x02_Socket, Q1 NTBLS0D8N08XTXG, Q2 NTBLS0D8N08XTXG, Q3 NTBLS0D8N08XTXG, Q6 BCP56, Q7 NTBLS0D8N08XTXG, U1 STM32F412RGTx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

Commit message: progress, also added footprints for redcube
Parts:
- removed J4: Conn_01x02_Socket, Connector_JST:JST_GH_SM02B-GHS-TB_1x02-1MP_P1.25mm_Horizontal
- added MP1: 7461117, Footprints-Symbols-Models:MP_Wurth_WP-RAFU_7461117, F.Cu at (155.1, 136.4)
- added MP2: 7461117, Footprints-Symbols-Models:MP_Wurth_WP-RAFU_7461117, F.Cu at (130.2, 136.5)
- added MP3: 7461090, Footprints-Symbols-Models:MP_Wurth_WP-BUCF_7461090, F.Cu at (181.5, 112.2)
- added MP4: 7461090, Footprints-Symbols-Models:MP_Wurth_WP-BUCF_7461090, F.Cu at (181.5, 61.4)
- added MP5: 7461090, Footprints-Symbols-Models:MP_Wurth_WP-BUCF_7461090, F.Cu at (156.5, 61.5)
- added R56: 100k, Resistor_SMD:R_0603_1608Metric, F.Cu at (69.2, 94.1)
- added TP1: TestPoint, TestPoint:TestPoint_Pad_2.0x2.0mm, F.Cu at (84.7, 61.7)
- added TP10: TestPoint, TestPoint:TestPoint_Pad_2.0x2.0mm, F.Cu at (84.7, 77.9)
- added TP2: TestPoint, TestPoint:TestPoint_Pad_2.0x2.0mm, F.Cu at (84.7, 65.8)
- added TP3: TestPoint, TestPoint:TestPoint_Pad_2.0x2.0mm, F.Cu at (84.7, 69.8)
- added TP4: TestPoint, TestPoint:TestPoint_Pad_2.0x2.0mm, F.Cu at (84.7, 73.8)
- added TP5: TestPoint, TestPoint:TestPoint_Bridge_Pitch2.54mm_Drill1.0mm, F.Cu at (84.7, 83.5)
- J1: footprint Connector_JST:JST_GH_BM04B-GHS-TBT_1x04-1MP_P1.25mm_Vertical -> Connector_JST:JST_ZH_B4B-ZR_1x04_P1.50mm_Vertical
- J2: footprint Connector_JST:JST_PHD_S24B-PHDSS_2x12_P2.00mm_Horizontal -> Connector_JST:JST_PHD_B24B-PHDSS_2x12_P2.00mm_Vertical
- J3: footprint Connector_JST:JST_EH_S13B-EH_1x13_P2.50mm_Horizontal -> Connector_JST:JST_EH_B13B-EH-A_1x13_P2.50mm_Vertical
- moved R62 182.6 mm to (233.3, 107.3)
- moved R64 182.6 mm to (233.3, 109.0)
- moved TH3 182.6 mm to (229.5, 109.5)
- moved TH1 122.0 mm to (159.0, 111.0)
- moved R3 105.9 mm to (115.8, 124.0), turned to -90 degrees
- moved R1 101.3 mm to (113.9, 124.0), turned to -90 degrees
- moved R2 100.2 mm to (110.7, 124.2), turned to -90 degrees
- moved J2 98.8 mm to (55.2, 144.1)
- moved C20 98.2 mm to (49.1, 74.0)
- moved C34 98.2 mm to (53.1, 74.0)
- moved C6 98.2 mm to (45.1, 74.0)
- moved R23 98.2 mm to (61.1, 74.0)
- moved R37 98.2 mm to (65.1, 74.0)
- moved R51 98.2 mm to (69.1, 74.0)
- moved R9 98.2 mm to (57.1, 74.0)
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Connections:
- C37 pad 1: /VDD1 -> /INPUT
- J2 pad 1: Net-(J2-Pin_1) -> GND
- J2 pad 11: Net-(J2-Pin_11) -> GND
- J2 pad 14: GND -> Net-(J2-Pin_14)
- J2 pad 16: GND -> Net-(J2-Pin_16)
- J2 pad 18: GND -> Net-(J2-Pin_18)
- J2 pad 20: GND -> Net-(J2-Pin_20)
- J2 pad 22: GND -> Net-(J2-Pin_22)
- J2 pad 24: GND -> Net-(J2-Pin_24)
- J2 pad 3: Net-(J2-Pin_3) -> GND
- J2 pad 5: Net-(J2-Pin_5) -> GND
- J2 pad 7: Net-(J2-Pin_7) -> GND
- J2 pad 9: Net-(J2-Pin_9) -> GND
- R33 pad 1: /VDD1 -> /INPUT
- R34 pad 2: Net-(J2-Pin_12) -> Net-(J2-Pin_24)
- R41 pad 2: Net-(J2-Pin_11) -> Net-(J2-Pin_22)
- R42 pad 2: Net-(J2-Pin_10) -> Net-(J2-Pin_20)
- R44 pad 2: Net-(J2-Pin_7) -> Net-(J2-Pin_14)
- R45 pad 2: Net-(J2-Pin_8) -> Net-(J2-Pin_16)
- R46 pad 2: Net-(J2-Pin_9) -> Net-(J2-Pin_18)
- R47 pad 2: Net-(J2-Pin_1) -> Net-(J2-Pin_2)
- R48 pad 2: Net-(J2-Pin_2) -> Net-(J2-Pin_4)
- R49 pad 2: Net-(J2-Pin_3) -> Net-(J2-Pin_6)
- R50 pad 2: Net-(J2-Pin_4) -> Net-(J2-Pin_8)
- R51 pad 2: Net-(J2-Pin_5) -> Net-(J2-Pin_10)
- R52 pad 2: Net-(J2-Pin_6) -> Net-(J2-Pin_12)
- R62 pad 1: /VCC -> /INPUT
- R64 pad 1: /VCC -> /INPUT
- U1 pad 12: unconnected-(U1-VSSA-Pad12) -> GND
- U1 pad 19: /VDD1 -> /INPUT
- U3 pad 1: /VDD1 -> /INPUT
- U4 pad 2: Net-(J2-Pin_8) -> Net-(J2-Pin_16)
- U4 pad 20: Net-(J2-Pin_12) -> Net-(J2-Pin_24)
- U4 pad 21: Net-(J2-Pin_11) -> Net-(J2-Pin_22)
- U4 pad 22: Net-(J2-Pin_10) -> Net-(J2-Pin_20)
- U4 pad 23: Net-(J2-Pin_9) -> Net-(J2-Pin_18)
- U4 pad 3: Net-(J2-Pin_7) -> Net-(J2-Pin_14)
- U4 pad 4: Net-(J2-Pin_6) -> Net-(J2-Pin_12)
- U4 pad 5: Net-(J2-Pin_5) -> Net-(J2-Pin_10)
- U4 pad 6: Net-(J2-Pin_4) -> Net-(J2-Pin_8)
- U4 pad 7: Net-(J2-Pin_3) -> Net-(J2-Pin_6)
- U4 pad 8: Net-(J2-Pin_2) -> Net-(J2-Pin_4)
- U4 pad 9: Net-(J2-Pin_1) -> Net-(J2-Pin_2)
- VR1 pad 5: /VDD1 -> /INPUT
Routing:
- net /DIODE+: track 0.00 -> 444.2 mm
- net /BAT+: track 0.00 -> 78.2 mm
- added copper zone on In1.Cu, net /BAT+
- added copper zone on In1.Cu, net GND
- added copper zone on In2.Cu, net GND
