File: electrical/BMS/BMS_vtest/BMS_vtest.kicad_sch (KiCad schematic)
At the start: 80 parts, among them Q1 NMOS, Q2 NPN, U2 BQ79612PAPRQ1, U3 CD74HC4067M, U4 STM32F103C6Tx

Commit message: oops most updated version ig (please check if my connectors are ok (i don't have a sense of direction), also i know one of them should be going on the back of the PCB)
Parts:
- removed Q1: NMOS, symbol Simulation_SPICE:NMOS
- removed Q2: NPN, symbol Simulation_SPICE:NPN
- removed U3: CD74HC4067M, Package_SO:SOIC-24W_7.5x15.4mm_P1.27mm, symbol 74xx:CD74HC4067M
- removed U4: STM32F103C6Tx, Package_QFP:LQFP-48_7x7mm_P0.5mm, symbol MCU_ST_STM32F1:STM32F103C6Tx
- added C36, C37, C38: 1u, Capacitor_SMD:C_0603_1608Metric, symbol Device:C
- added C39: 680n, Capacitor_SMD:C_0603_1608Metric, symbol Device:C
- added J1: Conn_01x04_Pin, Connector_JST:JST_GH_BM04B-GHS-TBT_1x04-1MP_P1.25mm_Vertical, symbol Connector:Conn_01x04_Pin
- added J2: Conn_02x12_Top_Bottom, Connector_JST:JST_PHD_S24B-PHDSS_2x12_P2.00mm_Horizontal, symbol Connector_Generic:Conn_02x12_Top_Bottom
- added J3: Conn_01x13_Socket, Connector_JST:JST_EH_S13B-EH_1x13_P2.50mm_Horizontal, symbol Connector:Conn_01x13_Socket
- added J4: Conn_01x02_Socket, Connector_JST:JST_GH_SM02B-GHS-TB_1x02-1MP_P1.25mm_Horizontal, symbol Connector:Conn_01x02_Socket
- added Q1, Q2, Q3, Q7: NTBLS0D8N08XTXG, Footprints-Symbols-Models:H-PSOF8L_100CU_ONS_OSI, symbol 2026-01-24_03-56-13:NTBLS0D8N08XTXG
- added Q6: BCP56, Package_TO_SOT_SMD:SOT-223-3_TabPin2, symbol Transistor_BJT:BCP56
- added R38: 0.1m, Resistor_SMD:R_0603_1608Metric, symbol Device:R
- added R39, R40, R55, R59: 10, Resistor_SMD:R_0603_1608Metric, symbol Device:R
- added R41, R42, R43, R44, R45, R46, R47, R48, R49, R50, R51, R52, R53, R62, R64: 10k, Resistor_SMD:R_0603_1608Metric, symbol Device:R
- added R54, R58: 100k, Resistor_SMD:R_0603_1608Metric, symbol Device:R
- added U1: STM32F412RGTx, Package_QFP:LQFP-64_10x10mm_P0.5mm, symbol MCU_ST_STM32F4:STM32F412RGTx
- added U3: ISO1044BD, Package_SO:SOIC-8_3.9x4.9mm_P1.27mm, symbol Interface_CAN_LIN:ISO1044BD
- added U4: CD74HC4067M, Package_SO:SOIC-24W_7.5x15.4mm_P1.27mm, symbol 74xx:CD74HC4067M
- added U5: PTPS48100QDGXRQ1, PTPS48100QDGXRQ1:VSSOP19_DGX_TEX, symbol TPS4810-Q1:PTPS48100QDGXRQ1
- added VR1: AP7366-33W5-7, Footprints-Symbols-Models:SOT95P285X140-5N, symbol AP7366-33W5-7:AP7366-33W5-7
- C1, C10, C11, C12, C13, C14, C15, C16, C17, C18, C19, C2, C20, C21, C22, C23, C24, C25, C26, C27, C28, C29, C3, C30, C31, C32, C33, C34, C35, C4, C5, C6, C7, C8, C9: footprint (none) -> Capacitor_SMD:C_0603_1608Metric
- R1, R10, R11, R12, R13, R14, R15, R16, R17, R18, R19, R2, R20, R21, R22, R23, R24, R25, R26, R27, R28, R29, R3, R30, R31, R32, R33, R34, R35, R36, R37, R4, R5, R6, R7, R8, R9, TH1, TH2, TH3: footprint (none) -> Resistor_SMD:R_0603_1608Metric
- U2: value BQ79612PAPRQ1 -> BQ79652PAPRQ1; footprint footprints:QFP_2PAPRQ1_TEX -> Footprints-Symbols-Models:QFP_2PAPRQ1_TEX
Connections:
- net AFE_RX: now also U1.22 (PA6)
- net AFE_TX: now also U1.23 (PA7)
- net AVDD: now also C36.1, R43.1, U4.24 (VCC), VR1.1 (IN)
- net CELL_1+: now also J3.12 (Pin_12)
- net CELL_10+: now also J3.3 (Pin_3)
- net CELL_11+: now also J3.2 (Pin_2)
- net CELL_12+: now also J3.1 (Pin_1)
- net CELL_2+: now also J3.11 (Pin_11)
- net CELL_3+: now also J3.10 (Pin_10)
- net CELL_4+: now also J3.9 (Pin_9)
- net CELL_5+: now also J3.8 (Pin_8)
- net CELL_6+: now also J3.7 (Pin_7)
- net CELL_7+: now also J3.6 (Pin_6)
- net CELL_8+: now also J3.5 (Pin_5)
- net GND: now also C35.1, R37.2, C36.2, C37.2, J2.13 (Pin_13), J2.14 (Pin_14), J2.15 (Pin_15), J2.16 (Pin_16), J2.17 (Pin_17), J2.18 (Pin_18), J2.19 (Pin_19), J2.20 (Pin_20), J2.21 (Pin_21), J2.22 (Pin_22), J2.23 (Pin_23), J2.24 (Pin_24), R38.2, R40.1, R53.2, U1.18 (VSS), U1.31 (VSS), U1.47 (VSS), U1.63 (VSS), U3.4 (GND1), U4.12 (GND), U4.15 (~{E}), U4.16 (I15), U4.17 (I14), U4.18 (I13), U4.19 (I12), U5.10 (SCP_TEST), U5.2 (INP2), U5.5 (*FLT), U5.6 (GND), U5.7 (CS_SEL), U5.8 (ISCP), U5.9 (TMR), VR1.2 (GND); no longer C35.2, R1.2, R3.2
- net GPIO2: now also U4.10 (S0); no longer C35.1, R34.1, R34.2, R35.1, R37.1, TH1.1, U2.51
- net GPIO3: now also U4.11 (S1); no longer R37.2, TH3.1
- net GPIO4: now also U4.14 (S2); no longer R35.2, R36.1, TH2.1
- net LDOIN: now also Q6.3 (E)
- net NPNB: now also Q6.1 (B)
- net VDD1: now also C37.1, U1.19 (VDD), U3.1 (VCC1), VR1.5 (OUT)
- net at C29.1, R30.1: now also Q6.2 (C), Q6.4 (C)
- net at U2.54: now also R37.1
- net at U2.55: now also R53.1
- net GPIO6: now reaches U2.56
- net GPIO6: now also R35.2, R36.1, TH2.1
- net GPIO5: now reaches U2.57
- net GPIO5: now also U4.13 (S3)
- net GPIO1: now reaches U2.61
- net GPIO1: now also U4.1 (COM)
- net NFAULT: now reaches U2.62
- net SRN: now reaches U2.63
- net SRN: now also C38.2, R40.2
- net SRP: now reaches U2.64
- net SRP: now also C38.1, R39.2
- net BAT renamed BAT+
- net BAT+: now also J4.1 (Pin_1), Q1.9, Q2.9, U5.1 (EN/UVLO), U5.17 (CS-), U5.18 (CS+), U5.20 (VS)
- net CELL_10- renamed CELL_9+
- net CELL_9+: now also J3.4 (Pin_4)
- new net: J2.8 (Pin_8), R45.2, U4.2 (I7)
- new net: J2.1 (Pin_1), R47.2, U4.9 (I0)
- new net: Q1.1, R54.2, R55.2
- new net: C39.2, U5.12 (BST)
- new net: R43.2, VR1.3 (EN)
- new net: J2.6 (Pin_6), R52.2, U4.4 (I5)
- new net: J2.10 (Pin_10), R42.2, U4.22 (I9)
- new net: J2.5 (Pin_5), R51.2, U4.5 (I4)
- new net: J2.11 (Pin_11), R41.2, U4.21 (I10)
- new net: J2.2 (Pin_2), R48.2, U4.8 (I1)
- new net: J1.1 (Pin_1), U3.7 (GND2)
- new net: J1.2 (Pin_2), U3.5 (CANL)
- new net: J1.3 (Pin_3), U3.6 (CANH)
- new net: J1.4 (Pin_4), U3.8 (VCC2)
- new net: J2.12 (Pin_12), R34.2, U4.20 (I11)
- new net: J2.3 (Pin_3), R49.2, U4.7 (I2)
- new net: J2.4 (Pin_4), R50.2, U4.6 (I3)
- new net: J2.7 (Pin_7), R44.2, U4.3 (I6)
- new net: J2.9 (Pin_9), R46.2, U4.23 (I8)
- new net: Q2.1, R58.2, R59.2
- new net BAT-: J4.2 (Pin_2)
- new net CELL_1-: J3.13 (Pin_13), R1.2, R3.2, R38.1, R39.1
- new net DIODE+: Q1.2, Q1.3, Q1.4, Q1.5, Q1.6, Q1.7, Q1.8, Q2.2, Q2.3, Q2.4, Q2.5, Q2.6, Q2.7, Q2.8, Q3.2, Q3.3, Q3.4, Q3.5, Q3.6, Q3.7, Q3.8, Q7.2, Q7.3, Q7.4, Q7.5, Q7.6, Q7.7, Q7.8
- new net G1PD: R55.1, R59.1, U5.14 (G1PD)
- new net G1PU: R54.1, R58.1, U5.15 (G1PI)
- new net G2: Q3.1, Q7.1, U5.11 (G2)
- new net INPUT: U1.14 (PA0), U5.3 (INP1)
- new net PA1: R62.2, TH1.1, U1.15 (PA1)
- new net PA2: R64.2, TH3.1, U1.16 (PA2)
- new net RXD: U1.41 (PA8), U3.3 (RXD)
- new net SRC: C39.1, Q3.9, Q7.9, U5.13 (SRC)
- new net TSREF: C35.2, R34.1, R35.1, R41.1, R42.1, R44.1, R45.1, R46.1, R47.1, R48.1, R49.1, R50.1, R51.1, R52.1, U2.51
- new net TXD: U1.42 (PA9), U3.2 (TXD)
- new net VCC: R62.1, R64.1
Other:
- note added: "CAN Transciever"
- note added: "Current Sense"
- note added: "LDO"
- note removed: "(STM) Load Switch"
- note removed: "MOSFET (2) Ambient Temperature (3) PCB Cell Balancing (4)"
- moved on the sheet: C1, C10, C11, C12, C13, C14, C15, C16, C17, C18, C19, C2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

Commit message: progress, also added footprints for redcube
Parts:
- removed J4: Conn_01x02_Socket, Connector_JST:JST_GH_SM02B-GHS-TB_1x02-1MP_P1.25mm_Horizontal, symbol Connector:Conn_01x02_Socket
- added MP1, MP2: 7461117, Footprints-Symbols-Models:MP_Wurth_WP-RAFU_7461117, symbol REDCUBE_Wurth_WP-RAFU:7461117
- added MP3, MP4, MP5: 7461090, Footprints-Symbols-Models:MP_Wurth_WP-BUCF_7461090, symbol REDCUBE_Wurth_WP-BUCF:7461090
- added R56: 100k, Resistor_SMD:R_0603_1608Metric, symbol Device:R
- added TP1, TP10, TP2, TP3, TP4: TestPoint, TestPoint:TestPoint_Pad_2.0x2.0mm, symbol Connector:TestPoint
- added TP5: TestPoint, TestPoint:TestPoint_Bridge_Pitch2.54mm_Drill1.0mm, symbol Connector:TestPoint
- J1: footprint Connector_JST:JST_GH_BM04B-GHS-TBT_1x04-1MP_P1.25mm_Vertical -> Connector_JST:JST_ZH_B4B-ZR_1x04_P1.50mm_Vertical
- J2: footprint Connector_JST:JST_PHD_S24B-PHDSS_2x12_P2.00mm_Horizontal -> Connector_JST:JST_PHD_B24B-PHDSS_2x12_P2.00mm_Vertical
- J3: footprint Connector_JST:JST_EH_S13B-EH_1x13_P2.50mm_Horizontal -> Connector_JST:JST_EH_B13B-EH-A_1x13_P2.50mm_Vertical
Connections:
- net VCC is gone; now on net INPUT: R62.1, R64.1
- net VDD1 is gone; now on net INPUT: C37.1, R33.1, U1.19 (VDD), U3.1 (VCC1), VR1.5 (OUT)
- net AFE_RX: now also TP2.1
- net AFE_TX: now also TP10.1
- net BAT+: now also MP1.1
- net DIODE+: now also MP3.1
- net GND: now also J2.1 (Pin_1), J2.11 (Pin_11), J2.3 (Pin_3), J2.5 (Pin_5), J2.7 (Pin_7), J2.9 (Pin_9), U1.12 (VSSA), MP2.1, MP5.1, R56.1, TP5.1; no longer J2.14 (Pin_14), J2.16 (Pin_16), J2.18 (Pin_18), J2.20 (Pin_20), J2.22 (Pin_22), J2.24 (Pin_24)
- net INPUT: now also R56.2, TP1.1
- net RXD: now also TP3.1
- net TXD: now also TP4.1
- net at R45.2, U4.2 (I7): now also J2.16 (Pin_16); no longer J2.8 (Pin_8)
- net at R47.2, U4.9 (I0): now also J2.2 (Pin_2); no longer J2.1 (Pin_1)
- net at R52.2, U4.4 (I5): now also J2.12 (Pin_12); no longer J2.6 (Pin_6)
- net at R42.2, U4.22 (I9): now also J2.20 (Pin_20); no longer J2.10 (Pin_10)
- net at R51.2, U4.5 (I4): now also J2.10 (Pin_10); no longer J2.5 (Pin_5)
- net at R41.2, U4.21 (I10): now also J2.22 (Pin_22); no longer J2.11 (Pin_11)
- net at R48.2, U4.8 (I1): now also J2.4 (Pin_4); no longer J2.2 (Pin_2)
- net at R34.2, U4.20 (I11): now also J2.24 (Pin_24); no longer J2.12 (Pin_12)
- net at R49.2, U4.7 (I2): now also J2.6 (Pin_6); no longer J2.3 (Pin_3)
- net at R50.2, U4.6 (I3): now also J2.8 (Pin_8); no longer J2.4 (Pin_4)
- net at R44.2, U4.3 (I6): now also J2.14 (Pin_14); no longer J2.7 (Pin_7)
- net at R46.2, U4.23 (I8): now also J2.18 (Pin_18); no longer J2.9 (Pin_9)
- new net BMS+: MP4.1
Other:
- note added: "BMS IC Cell Temperatures"
- note added: "BMS IC Current Balancing"
- note added: "Connectors"
- note added: "Gate Driver NMOS"
- note added: "STM32 ADC Ambient & Gate Driver MOSFETs"
- moved on the sheet: C1, C10, C11, C12, C13, C14, C15, C16, C17, C18, C19, C2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
